Commit message: Renamed files and folders to match conventions (xacro files) Fixed parenthesis issues in util.urdf.xacro Fixed CMakeLists.txt in lwr_simulation to get lwr_controller installed

File: lwr_description/robots/kuka_lwr_arm.urdf.xacro (robot description, xacro)
@@ -1,7 +1,7 @@
 <?xml version="1.0"?>
 <robot name="lwr" xmlns:xacro="http://www.ros.org/wiki/xacro" >
-  <xacro:include filename="$(find lwr_defs)/defs/kuka_lwr_arm_defs.xml"/>
-  <xacro:include filename="$(find lwr_defs)/defs/gazebo_defs.xml"/>
-  <xacro:include filename="$(find lwr_defs)/defs/materials.xml"/>
+  <xacro:include filename="$(find lwr_description)/urdf/lwr.urdf.xacro"/>
+  <xacro:include filename="$(find lwr_description)/urdf/lwr_gazebo.urdf.xacro"/>
+  <xacro:include filename="$(find lwr_description)/urdf/materials.urdf.xacro"/>
    <link name="world" />
   <joint name="arm_world_joint" type="fixed">

File: lwr_description/urdf/lwr.urdf.xacro (robot description, xacro)
@@ -4,5 +4,5 @@
        xmlns:interface="http://playerstage.sourceforge.net/gazebo/xmlschema/#interface"
        xmlns:xacro="http://www.ros.org/wiki/xacro">
-  <xacro:include filename="$(find lwr_defs)/defs/util_defs.xml"/>
+  <xacro:include filename="$(find lwr_description)/urdf/util.urdf.xacro"/>
   <property name="arm_elem_base_mass" value="2.0"/>
   <property name="arm_elem_link_mass" value="2.0"/>
@@ -28,5 +28,5 @@
         <origin xyz="0 0 0" rpy="0 0 0"/>
         <geometry>
-          <mesh filename="package://lwr_defs/meshes/lwr/base.STL"/>
+          <mesh filename="package://lwr_description/meshes/lwr/base.STL"/>
         </geometry>
         <material name="Orange"/>
@@ -35,5 +35,5 @@
         <origin xyz="0 0 0.055" rpy="0 0 ${M_PI}"/>
         <geometry>
-<!--          <mesh filename="package://lwr_defs/meshes/lwr/convex/arm_base_convex.stl"/> -->
+<!--          <mesh filename="package://lwr_description/meshes/lwr/convex/arm_base_convex.stl"/> -->
           <cylinder radius="0.07" length="0.11"/>
         </geometry>
@@ -69,13 +69,13 @@
         <origin xyz="0 0 -0.008" rpy="0 0 0"/>
         <geometry>
-          <mesh filename="package://lwr_defs/meshes/lwr/link_1.STL"/>
-        </geometry>
-        <material name="Orange"/>
-      </visual>
-<!--
-      <collision>
-        <origin xyz="0 0 0" rpy="0 0 0"/>
-        <geometry>
-          <mesh filename="package://lwr_defs/meshes/lwr/convex/arm_segment_a_convex.stl"/>
+          <mesh filename="package://lwr_description/meshes/lwr/link_1.STL"/>
+        </geometry>
+        <material name="Orange"/>
+      </visual>
+<!--
+      <collision>
+        <origin xyz="0 0 0" rpy="0 0 0"/>
+        <geometry>
+          <mesh filename="package://lwr_description/meshes/lwr/convex/arm_segment_a_convex.stl"/>
         </geometry>
       </collision>
@@ -132,5 +132,5 @@
         <origin xyz="0 0 0.0" rpy="0 0 0"/>
         <geometry>
-          <mesh filename="package://lwr_defs/meshes/lwr/link_2.STL"/>
+          <mesh filename="package://lwr_description/meshes/lwr/link_2.STL"/>
         </geometry>
         <material name="Orange"/>
@@ -140,5 +140,5 @@
         <origin xyz="0 0 0.2" rpy="${M_PI} 0 0"/>
         <geometry>
-          <mesh filename="package://lwr_defs/meshes/lwr/convex/arm_segment_b_convex.stl"/>
+          <mesh filename="package://lwr_description/meshes/lwr/convex/arm_segment_b_convex.stl"/>
         </geometry>
       </collision>
@@ -195,5 +195,5 @@
         <origin xyz="0 0 -0.008" rpy="0 0 0"/>
         <geometry>
-          <mesh filename="package://lwr_defs/meshes/lwr/link_3.STL"/>
+          <mesh filename="package://lwr_description/meshes/lwr/link_3.STL"/>
         </geometry>
         <material name="Orange"/>
@@ -203,5 +203,5 @@
         <origin xyz="0 0 0" rpy="0 0 ${M_PI}"/>
         <geometry>
-          <mesh filename="package://lwr_defs/meshes/lwr/convex/arm_segment_a_convex.stl"/>
+          <mesh filename="package://lwr_description/meshes/lwr/convex/arm_segment_a_convex.stl"/>
         </geometry>
       </collision>
@@ -258,5 +258,5 @@
         <origin xyz="0 0 0.0" rpy="0 0 0"/>
         <geometry>
-          <mesh filename="package://lwr_defs/meshes/lwr/link_4.STL"/>
+          <mesh filename="package://lwr_description/meshes/lwr/link_4.STL"/>
         </geometry>
         <material name="Orange"/>
@@ -266,5 +266,5 @@
         <origin xyz="0 0 0.2" rpy="0 ${M_PI} 0"/>
         <geometry>
-          <mesh filename="package://lwr_defs/meshes/lwr/convex/arm_segment_b_convex.stl"/>
+          <mesh filename="package://lwr_description/meshes/lwr/convex/arm_segment_b_convex.stl"/>
         </geometry>
       </collision>
@@ -321,13 +321,13 @@
         <origin xyz="0 0 -0.008" rpy="0 0 0"/>
         <geometry name="${name}_arm_5_geom">
-          <mesh filename="package://lwr_defs/meshes/lwr/link_5.STL"/>
-        </geometry>
-        <material name="Orange"/>
-      </visual>
-<!--
-      <collision>
-        <origin xyz="0 0 0" rpy="0 0 0"/>
-        <geometry>
-          <mesh filename="package://lwr_defs/meshes/lwr/convex/arm_segment_last_convex.stl"/>
+          <mesh filename="package://lwr_description/meshes/lwr/link_5.STL"/>
+        </geometry>
+        <material name="Orange"/>
+      </visual>
+<!--
+      <collision>
+        <origin xyz="0 0 0" rpy="0 0 0"/>
+        <geometry>
+          <mesh filename="package://lwr_description/meshes/lwr/convex/arm_segment_last_convex.stl"/>
         </geometry>
       </collision>
@@ -383,5 +383,5 @@
         <origin xyz="0 0 0" rpy="0 0 0"/>
         <geometry>
-          <mesh filename="package://lwr_defs/meshes/lwr/link_6.STL"/>
+          <mesh filename="package://lwr_description/meshes/lwr/link_6.STL"/>
         </geometry>
         <material name="Grey"/>
@@ -390,5 +390,5 @@
         <origin xyz="0 0 0" rpy="0 0 0"/>
         <geometry>
-          <mesh filename="package://lwr_defs/meshes/lwr/convex/arm_wrist_convex.stl"/>
+          <mesh filename="package://lwr_description/meshes/lwr/convex/arm_wrist_convex.stl"/>
         </geometry>
       </collision>
@@ -425,5 +425,5 @@
         <origin xyz="0 0 0" rpy="0 0 0"/>
         <geometry>
-          <mesh filename="package://lwr_defs/meshes/lwr/link_7.STL"/>
+          <mesh filename="package://lwr_description/meshes/lwr/link_7.STL"/>
         </geometry>
         <material name="Grey"/>

File: lwr_description/urdf/util.urdf.xacro (robot description, xacro)
@@ -10,14 +10,14 @@
      -->
   <macro name="cuboid_inertia_def" params="width height length mass">
-    <inertia ixx="${mass * (height * height + length * length) / 12)}"
-             iyy="${mass * (width * width + length * length) / 12)}"
-             izz="${mass * (width * width + height * height) / 12)}"
+    <inertia ixx="${mass * (height * height + length * length) / 12}"
+             iyy="${mass * (width * width + length * length) / 12}"
+             izz="${mass * (width * width + height * height) / 12}"
              ixy="0" iyz="0" ixz="0"/>
   </macro>
   <!-- length is along the y-axis! -->
   <macro name="cylinder_inertia_def" params="radius length mass">
-    <inertia ixx="${mass * (3 * radius * radius + length * length) / 12)}"
-             iyy="${mass * radius* radius / 2)}"
-             izz="${mass * (3 * radius * radius + length * length) / 12)}"
+    <inertia ixx="${mass * (3 * radius * radius + length * length) / 12}"
+             iyy="${mass * radius*radius / 2}"
+             izz="${mass * (3 * radius * radius + length * length) / 12}"
              ixy="0" iyz="0" ixz="0"/>
   </macro>

Commit message: Migrated to newer plugin xacro description with parameters

File: lwr_description/robots/kuka_lwr_arm.urdf.xacro (robot description, xacro)
@@ -34,3 +34,4 @@
     <origin xyz="0 0 1.1" rpy="0 0 0"/>
   </xacro:kuka_lwr_arm>
+  <xacro:lwr_arm_gazebo_controller namespace="" prefix="lwr" port="49938"/>
 </robot>

File: lwr_description/urdf/lwr.urdf.xacro (robot description, xacro)
@@ -16,7 +16,7 @@
       <insert_block name="origin"/>
       <parent link="${parent}_link"/>
-      <child link="calib_${name}_arm_base_link"/>
-    </joint>
-    <link name="calib_${name}_arm_base_link">
+      <child link="${name}_arm_base_link"/>
+    </joint>
+    <link name="${name}_arm_base_link">
       <inertial>
         <mass value="${arm_elem_base_mass}"/>
@@ -56,5 +56,5 @@
                          k_velocity="30"/>
       <dynamics damping="1.0"/>
-      <parent link="calib_${name}_arm_base_link"/>
+      <parent link="${name}_arm_base_link"/>
       <child link="${name}_arm_1_link"/>
     </joint>

File: lwr_description/urdf/lwr_gazebo.urdf.xacro (robot description, xacro)
@@ -1,18 +1,35 @@
-<robot xmlns:sensor="http://playerstage.sourceforge.net/gazebo/xmlschema/#sensor"
-       xmlns:controller="http://playerstage.sourceforge.net/gazebo/xmlschema/#controller"
-       xmlns:interface="http://playerstage.sourceforge.net/gazebo/xmlschema/#interface">
-  <gazebo>
-    <plugin name="lwr_controller" filename="liblwr_controller.so">
-      <alwaysOn>true</alwaysOn>
-      <robotPrefix>lwr</robotPrefix>
-      <remotePort>49938</remotePort>
-      <lwr_arm_0_joint>0.0</lwr_arm_0_joint>
-      <lwr_arm_1_joint>0.7</lwr_arm_1_joint>
-      <lwr_arm_2_joint>0.0</lwr_arm_2_joint>
-      <lwr_arm_3_joint>-0.7</lwr_arm_3_joint>
-      <lwr_arm_4_joint>0.7</lwr_arm_4_joint>
-      <lwr_arm_5_joint>0.7</lwr_arm_5_joint>
-      <lwr_arm_6_joint>0.7</lwr_arm_6_joint>
-    </plugin>
-  </gazebo>
+<?xml version="1.0"?>
+<robot xmlns:xacro="http://www.ros.org/wiki/xacro">
+	<!-- namespace must be set up according to launch file namespace -->
+	<!-- port is the port number for the FRI UDP connection (be aware that port+1 is also used) -->
+	<xacro:macro name="lwr_arm_gazebo_controller" params="namespace port prefix gravity_dir:=^|'0 0 -9.81'
+		                                                    payload_mass:=^|0.0 payload_cog:=^|'0 0 0'">
+		<xacro:property name="prefix_"  value="${prefix + '_' if prefix else ''}" />
+		<gazebo>
+			<plugin name="${prefix_}lwr_arm_controller" filename="liblwr_controller.so">
+				<alwaysOn>true</alwaysOn>
+				<robotPrefix>${prefix}</robotPrefix>
+				<robotNamespace>${namespace}</robotNamespace>
+				<remotePort>${port}</remotePort>
+				<baseLink>${prefix_}arm_base_link</baseLink>
+				<!-- p<toolLink>${prefix_}tool_mount</toolLink>-->
+				<xacro:if value="${gravity_dir not in ['','-']}" >
+					<gravityDirection>${gravity_dir}</gravityDirection>
+				</xacro:if>
+				<xacro:if value="${payload_mass not in ['','-']}" >
+					<payloadMass>${payload_mass}</payloadMass>
+				</xacro:if>
+				<xacro:if value="${payload_cog not in ['','-']}" >
+					<payloadCOG>${payload_cog}</payloadCOG>
+				</xacro:if>
+				<xacro:element xacro:name="${prefix_}arm_0_joint">0</xacro:element>
+				<xacro:element xacro:name="${prefix_}arm_1_joint">0</xacro:element>
+				<xacro:element xacro:name="${prefix_}arm_2_joint">0</xacro:element>
+				<xacro:element xacro:name="${prefix_}arm_3_joint">0</xacro:element>
+				<xacro:element xacro:name="${prefix_}arm_4_joint">0</xacro:element>
+				<xacro:element xacro:name="${prefix_}arm_5_joint">0</xacro:element>
+				<xacro:element xacro:name="${prefix_}arm_6_joint">0</xacro:element>
+			</plugin>
+		</gazebo>
+	</xacro:macro>
 </robot>
