Commit message: Moved meshes and fixed authorship

File: lwr_description/robots/kuka_lwr_arm.urdf.xacro (robot description, xacro)
@@ -31,7 +31,11 @@
     </collision>
   </link>
-  <xacro:kuka_lwr_arm parent="world" name="lwr" right="1">
+  <!-- First (shoulder) element of the arm. Fixed to its parent. -->
+  <joint name="world_lwr_arm_base_joint" type="fixed">
     <origin xyz="0 0 1.1" rpy="0 0 0"/>
-  </xacro:kuka_lwr_arm>
+    <parent link="world_link"/>
+    <child link="lwr_arm_base_link"/>
+  </joint>
+  <xacro:kuka_lwr_arm name="lwr_" />
   <xacro:lwr_arm_gazebo_controller namespace="" prefix="lwr" port="49938"/>
 </robot>

File: lwr_description/urdf/lwr.urdf.xacro (robot description, xacro)
@@ -1,25 +1,21 @@
 <?xml version="1.0"?>
-<robot xmlns:sensor="http://playerstage.sourceforge.net/gazebo/xmlschema/#sensor"
-       xmlns:controller="http://playerstage.sourceforge.net/gazebo/xmlschema/#controller"
-       xmlns:interface="http://playerstage.sourceforge.net/gazebo/xmlschema/#interface"
-       xmlns:xacro="http://www.ros.org/wiki/xacro">
+<robot xmlns:xacro="http://www.ros.org/wiki/xacro"
+		 xmlns:sensor="http://playerstage.sourceforge.net/gazebo/xmlschema/#sensor"
+		 xmlns:controller="http://playerstage.sourceforge.net/gazebo/xmlschema/#controller"
+       xmlns:interface="http://playerstage.sourceforge.net/gazebo/xmlschema/#interface">
   <xacro:include filename="$(find lwr_description)/urdf/util.urdf.xacro"/>
-  <property name="arm_elem_base_mass" value="2.0"/>
-  <property name="arm_elem_link_mass" value="2.0"/>
-  <property name="arm_elem_end_link_mass" value="2.0"/>
-  <property name="arm_elem_ball_link_mass" value="2.0"/>
-  <property name="arm_velocity_scale_factor" value="1"/>
-  <!-- right is either 1 (for right arm) or -1 (for left arm) -->
-  <macro name="kuka_lwr_arm" params="parent name right *origin">
-    <!-- First (shoulder) element of the arm. Fixed to its parent. -->
-    <joint name="${parent}_${name}_arm_base_joint" type="fixed">
-      <insert_block name="origin"/>
-      <parent link="${parent}_link"/>
-      <child link="${name}_arm_base_link"/>
-    </joint>
-    <link name="${name}_arm_base_link">
+  <xacro:property name="arm_elem_base_mass" value="1.2"/>
+  <xacro:property name="arm_elem_link_mass" value="2.0"/>
+  <xacro:property name="arm_elem_ball_link_mass" value="1.0"/>
+  <xacro:property name="arm_elem_end_link_mass" value="0.2"/>
+  <xacro:property name="safety_controller_k_pos" value="100" />
+  <xacro:property name="safety_controller_k_vel" value="2" />
+  <xacro:property name="joint_damping_factor" value="1.0" />
+  <xacro:property name="arm_velocity_scale_factor" value="1"/>
+  <xacro:macro name="kuka_lwr_arm" params="name">
+    <link name="${name}arm_base_link">
       <inertial>
         <mass value="${arm_elem_base_mass}"/>
-        <origin xyz="0 0 0.055"/>
+        <origin xyz="0 0 0.055" rpy="0 0 0"/>
         <cylinder_inertia_def radius="0.06" length="0.11"
                               mass="${arm_elem_base_mass}"/>
@@ -28,420 +24,352 @@
         <origin xyz="0 0 0" rpy="0 0 0"/>
         <geometry>
-          <mesh filename="package://lwr_description/meshes/lwr/base.STL"/>
-        </geometry>
-        <material name="Orange"/>
-      </visual>
-      <collision>
-        <origin xyz="0 0 0.055" rpy="0 0 ${M_PI}"/>
-        <geometry>
-<!--          <mesh filename="package://lwr_description/meshes/lwr/convex/arm_base_convex.stl"/> -->
-          <cylinder radius="0.07" length="0.11"/>
-        </geometry>
-      </collision>
-    </link>
-<!--
-    <gazebo reference="calib_${name}_arm_base_link">
-      <turnGravityOff>false</turnGravityOff>
-    </gazebo>
--->
-    <!-- Second segment of the arm. Joint along z-axis -->
-    <joint name="${name}_arm_0_joint" type="revolute">
+          <mesh scale="100 100 100"
+					 filename="package://lwr_description/meshes/arm_base.dae"/>
+        </geometry>
+        <material name="Orange"/>
+      </visual>
+      <collision>
+        <origin xyz="0 0 0.01" rpy="0 0 0"/>
+        <geometry>
+          <mesh filename="package://lwr_description/meshes/convex/arm_base_convex.stl" scale="0.9 0.9 0.9"/>
+        </geometry>
+      </collision>
+    </link>
+    <gazebo reference="${name}arm_base_link">
+      <!--<material value="kuka-lwr.material"/>-->
+    </gazebo>
+    <joint name="${name}arm_0_joint" type="revolute">
       <origin xyz="0 0 0.11" rpy="0 0 0"/>
       <axis xyz="0 0 1"/>
-      <limit lower="${-170 * M_PI / 180}" upper="${170 * M_PI / 180}"
-             effort="204" velocity="${arm_velocity_scale_factor * 110 * M_PI / 180}" />
-      <safety_controller soft_lower_limit="${-168 * M_PI / 180}"
-                         soft_upper_limit="${168 * M_PI / 180}"
-                         k_position="30"
-                         k_velocity="30"/>
-      <dynamics damping="1.0"/>
-      <parent link="${name}_arm_base_link"/>
-      <child link="${name}_arm_1_link"/>
-    </joint>
-    <link name="${name}_arm_1_link">
-      <inertial>
-        <mass value="${arm_elem_link_mass}"/>
-        <origin rpy="0 0 0" xyz="0 -0.06 0.130"/>
-        <cuboid_inertia_def length="0.12" width="0.06" height="0.260"
-                            mass="${arm_elem_link_mass}"/>
-      </inertial>
-      <visual>
-        <origin xyz="0 0 -0.008" rpy="0 0 0"/>
-        <geometry>
-          <mesh filename="package://lwr_description/meshes/lwr/link_1.STL"/>
-        </geometry>
-        <material name="Orange"/>
-      </visual>
-<!--
-      <collision>
-        <origin xyz="0 0 0" rpy="0 0 0"/>
-        <geometry>
-          <mesh filename="package://lwr_description/meshes/lwr/convex/arm_segment_a_convex.stl"/>
-        </geometry>
-      </collision>
- -->
-      <collision>
-        <origin xyz="0 0 0.0" rpy="0 0 0"/>
-        <geometry>
-          <sphere radius="0.07"/>
-        </geometry>
-      </collision>
-      <collision>
-        <origin xyz="0 -0.06 0.2" rpy="0 0 0"/>
-        <geometry>
-          <sphere radius="0.07"/>
-        </geometry>
-      </collision>
-      <collision>
-        <origin xyz="0 -0.03 0.1" rpy="0.291 0 0"/>
-        <geometry>
-          <cylinder radius="0.07" length="0.208"/>
-        </geometry>
-      </collision>
-    </link>
-    <gazebo reference="${name}_arm_1_link">
-      <gravity>false</gravity>
-    </gazebo>
-    <transmission name="${name}_arm_0_trans" type="SimpleTransmission">
-      <actuator name="${name}_arm_0_motor"/>
-      <joint name="${name}_arm_0_joint"/>
-      <mechanicalReduction>1.0</mechanicalReduction>
-    </transmission>
-    <!-- Third segment of the arm. Joint along y-axis -->
-    <joint name="${name}_arm_1_joint" type="revolute">
-      <origin xyz="0 0 0.2005" rpy="0 0 0"/>
-      <axis xyz="0 1 0"/>
-      <limit lower="${-120 * M_PI / 180}" upper="${120 * M_PI / 180}"
-             effort="306" velocity="${arm_velocity_scale_factor * 110 * M_PI / 180}" />
-      <safety_controller soft_lower_limit="${-118 * M_PI / 180}"
-                         soft_upper_limit="${118 * M_PI / 180}"
-                         k_position="30"
-                         k_velocity="30"/>
-      <dynamics damping="1.0" friction="10"/>
-      <parent link="${name}_arm_1_link"/>
-      <child link="${name}_arm_2_link"/>
-    </joint>
-    <link name="${name}_arm_2_link">
-      <inertial>
-        <mass value="${arm_elem_link_mass}"/>
-        <origin rpy="0 0 0" xyz="0 0.06 ${0.130 - 0.06}"/>
-        <cuboid_inertia_def length="0.12" width="0.06" height="0.260"
-                            mass="${arm_elem_link_mass}"/>
-      </inertial>
-      <visual>
-        <origin xyz="0 0 0.0" rpy="0 0 0"/>
-        <geometry>
-          <mesh filename="package://lwr_description/meshes/lwr/link_2.STL"/>
-        </geometry>
-        <material name="Orange"/>
-      </visual>
-<!--
-      <collision>
-        <origin xyz="0 0 0.2" rpy="${M_PI} 0 0"/>
-        <geometry>
-          <mesh filename="package://lwr_description/meshes/lwr/convex/arm_segment_b_convex.stl"/>
-        </geometry>
-      </collision>
--->
-      <collision>
-        <origin xyz="0 0 0.2" rpy="0 0 0"/>
-        <geometry>
-          <sphere radius="0.07"/>
-        </geometry>
-      </collision>
-      <collision>
-        <origin xyz="0 0.06 0.0" rpy="0 0 0"/>
-        <geometry>
-          <sphere radius="0.07"/>
-        </geometry>
-      </collision>
-      <collision>
-        <origin xyz="0 0.03 0.1" rpy="0.291 0 0"/>
-        <geometry>
-          <cylinder radius="0.07" length="0.208"/>
-        </geometry>
-      </collision>
-    </link>
-    <gazebo reference="${name}_arm_2_link">
-      <gravity>false</gravity>
-    </gazebo>
-    <transmission name="${name}_arm_1_trans" type="SimpleTransmission">
-      <actuator name="${name}_arm_1_motor"/>
-      <joint name="${name}_arm_1_joint"/>
-      <mechanicalReduction>1.0</mechanicalReduction>
-    </transmission>
-    <!-- Fourth element of the arm. z-axis -->
-    <joint name="${name}_arm_2_joint" type="revolute">
+      <limit lower="${-170 * pi / 180}" upper="${170 * pi / 180}"
+             effort="204" velocity="${arm_velocity_scale_factor * 110 * pi / 180}" />
+      <safety_controller soft_lower_limit="${-168 * pi / 180}"
+                         soft_upper_limit="${168 * pi / 180}"
+                         k_position="${safety_controller_k_pos}"
+                         k_velocity="${safety_controller_k_vel}"/>
+      <dynamics damping="${joint_damping_factor*5.0}"/>
+      <parent link="${name}arm_base_link"/>
+      <child link="${name}arm_1_link"/>
+    </joint>
+    <gazebo reference="${name}arm_0_joint">
+      <provideFeedback>1</provideFeedback>
+      <implicitSpringDamper>1</implicitSpringDamper>
+    </gazebo>
+    <transmission name="${name}arm_0_trans" type="SimpleTransmission">
+      <actuator name="${name}arm_0_motor"/>
+      <joint name="${name}arm_0_joint"/>
+      <mechanicalReduction>1.0</mechanicalReduction>
+    </transmission>
+    <link name="${name}arm_1_link">
+      <inertial>
+        <mass value="${arm_elem_link_mass}"/>
+        <origin rpy="0 0 0" xyz="0 0 0.130"/>
+        <cuboid_inertia_def length="0.260" width="0.06" height="0.12"
+                            mass="${arm_elem_link_mass}"/>
+      </inertial>
+      <visual>
+        <origin xyz="0 0 0" rpy="0 0 ${pi}"/>
+        <geometry>
+          <mesh scale="100 100 100"  filename="package://lwr_description/meshes/arm_segment_a.dae"/>
+        </geometry>
+        <material name="Orange"/>
+      </visual>
+      <collision>
+        <origin xyz="0 0 0" rpy="0 0 ${pi}"/>
+        <geometry>
+          <mesh filename="package://lwr_description/meshes/convex/arm_segment_a_convex.stl" scale="1.0 1.0 1.0"/>
+        </geometry>
+      </collision>
+    </link>
+    <gazebo reference="${name}arm_1_link">
+      <!--<material value="kuka-lwr.material"/>-->
+    </gazebo>
+    <joint name="${name}arm_1_joint" type="revolute">
+      <origin xyz="0 0 0.20" rpy="0 0 0"/>
+      <axis xyz="0 -1 0"/>
+      <limit lower="${-120 * pi / 180}" upper="${120 * pi / 180}"
+             effort="306" velocity="${arm_velocity_scale_factor * 110 * pi / 180}" />
+      <safety_controller soft_lower_limit="${-118 * pi / 180}"
+                         soft_upper_limit="${118 * pi / 180}"
+                         k_position="${safety_controller_k_pos}"
+                         k_velocity="${safety_controller_k_vel}"/>
+      <dynamics damping="${joint_damping_factor*5.0}"/>
+      <parent link="${name}arm_1_link"/>
+      <child link="${name}arm_2_link"/>
+    </joint>
+    <gazebo reference="${name}arm_1_joint">
+      <provideFeedback>1</provideFeedback>
+      <implicitSpringDamper>1</implicitSpringDamper>
+    </gazebo>
+    <transmission name="${name}arm_1_trans" type="pr2_mechanism_model/SimpleTransmission">
+      <actuator name="${name}arm_1_motor"/>
+      <joint name="${name}arm_1_joint"/>
+      <mechanicalReduction>1.0</mechanicalReduction>
+    </transmission>
+    <link name="${name}arm_2_link">
+      <inertial>
+        <mass value="${arm_elem_link_mass}"/>
+        <origin rpy="0 0 0" xyz="0 -0.06 ${0.130 - 0.06}"/>
+        <cuboid_inertia_def length="0.260" width="0.06" height="0.12"
+                            mass="${arm_elem_link_mass}"/>
+      </inertial>
+      <visual>
+        <origin xyz="0 0 0.2" rpy="${pi} 0 ${pi}"/>
+        <geometry>
+          <mesh scale="100 100 100"
+					 filename="package://lwr_description/meshes/arm_segment_b.dae"/>
+        </geometry>
+        <material name="Orange"/>
+      </visual>
+      <collision>
+        <origin xyz="0 0 0.2" rpy="${pi} 0 ${pi}"/>
+        <geometry>
+          <mesh filename="package://lwr_description/meshes/convex/arm_segment_b_convex.stl" scale="1.0 1.0 1.0"/>
+        </geometry>
+      </collision>
+    </link>
+    <gazebo reference="${name}arm_2_link">
+      <!--<material value="kuka-lwr.material"/>-->
+    </gazebo>
+    <joint name="${name}arm_2_joint" type="revolute">
       <origin xyz="0 0 0.20" rpy="0 0 0"/>
       <axis xyz="0 0 1"/>
-      <limit lower="${-170 * M_PI / 180}" upper="${170 * M_PI / 180}"
-             effort="204" velocity="${arm_velocity_scale_factor * 130 * M_PI / 180}" />
-      <safety_controller soft_lower_limit="${-168 * M_PI / 180}"
-                         soft_upper_limit="${168 * M_PI / 180}"
-                         k_position="30"
-                         k_velocity="30"/>
-      <dynamics damping="1.0"/>
-      <parent link="${name}_arm_2_link"/>
-      <child link="${name}_arm_3_link"/>
-    </joint>
-    <link name="${name}_arm_3_link">
-      <inertial>
-        <mass value="${arm_elem_link_mass}"/>
-        <origin rpy="0 0 0" xyz="0 0.06 0.130"/>
-        <cuboid_inertia_def length="0.12" width="0.06" height="0.260"
-                            mass="${arm_elem_link_mass}"/>
-      </inertial>
-      <visual>
-        <origin xyz="0 0 -0.008" rpy="0 0 0"/>
-        <geometry>
-          <mesh filename="package://lwr_description/meshes/lwr/link_3.STL"/>
-        </geometry>
-        <material name="Orange"/>
-      </visual>
-<!--
-      <collision>
-        <origin xyz="0 0 0" rpy="0 0 ${M_PI}"/>
-        <geometry>
-          <mesh filename="package://lwr_description/meshes/lwr/convex/arm_segment_a_convex.stl"/>
-        </geometry>
-      </collision>
--->
-      <collision>
-        <origin xyz="0 0 0.0" rpy="0 0 0"/>
-        <geometry>
-          <sphere radius="0.07"/>
-        </geometry>
-      </collision>
-      <collision>
-        <origin xyz="0 0.06 0.2" rpy="0 0 0"/>
-        <geometry>
-          <sphere radius="0.07"/>
-        </geometry>
-      </collision>
-      <collision>
-        <origin xyz="0 0.03 0.1" rpy="-0.291 0 0"/>
-        <geometry>
-          <cylinder radius="0.07" length="0.208"/>
-        </geometry>
-      </collision>
-    </link>
-    <gazebo reference="${name}_arm_3_link">
-      <gravity>false</gravity>
-    </gazebo>
-    <transmission name="${name}_arm_2_trans" type="SimpleTransmission">
-      <actuator name="${name}_arm_2_motor"/>
-      <joint name="${name}_arm_2_joint"/>
-      <mechanicalReduction>1.0</mechanicalReduction>
-    </transmission>
-    <!-- fifth element of the arm. x-axis -->
-    <joint name="${name}_arm_3_joint" type="revolute">
+      <limit lower="${-170 * pi / 180}" upper="${170 * pi / 180}"
+             effort="204" velocity="${arm_velocity_scale_factor * 130 * pi / 180}" />
+      <safety_controller soft_lower_limit="${-168 * pi / 180}"
+                         soft_upper_limit="${168 * pi / 180}"
+                         k_position="${safety_controller_k_pos}"
+                         k_velocity="${safety_controller_k_vel}"/>
+      <dynamics damping="${joint_damping_factor*3.0}"/>
+      <parent link="${name}arm_2_link"/>
+      <child link="${name}arm_3_link"/>
+    </joint>
+    <gazebo reference="${name}arm_2_joint">
+      <provideFeedback>1</provideFeedback>
+      <implicitSpringDamper>1</implicitSpringDamper>
+    </gazebo>
+    <transmission name="${name}arm_2_trans" type="SimpleTransmission">
+      <actuator name="${name}arm_2_motor"/>
+      <joint name="${name}arm_2_joint"/>
+      <mechanicalReduction>1.0</mechanicalReduction>
+    </transmission>
+    <link name="${name}arm_3_link">
+      <inertial>
+        <mass value="${arm_elem_link_mass}"/>
+        <origin rpy="0 0 0" xyz="0 -0.06 0.130"/>
+        <cuboid_inertia_def length="0.260" width="0.06" height="0.12"
+                            mass="${arm_elem_link_mass}"/>
+      </inertial>
+      <visual>
+        <origin xyz="0 0 0" rpy="0 0 0"/>
+        <geometry>
+          <mesh scale="100 100 100"
+					 filename="package://lwr_description/meshes/arm_segment_a.dae"/>
+        </geometry>
+        <material name="Orange"/>
+      </visual>
+      <collision>
+        <origin xyz="0 0 0" rpy="0 0 0"/>
+        <geometry>
+          <mesh filename="package://lwr_description/meshes/convex/arm_segment_a_convex.stl" scale="1.0 1.0 1.0"/>
+        </geometry>
+      </collision>
+    </link>
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
File: lwr_description/urdf/util.urdf.xacro (robot description, xacro)
@@ -1,24 +1,20 @@
 <?xml version="1.0"?>
-<robot xmlns:xacro="http://www.ros.org/wiki/xacro"
-       xmlns:sensor="http://playerstage.sourceforge.net/gazebo/xmlschema/#sensor"
-       xmlns:controller="http://playerstage.sourceforge.net/gazebo/xmlschema/#controller"
-       xmlns:interface="http://playerstage.sourceforge.net/gazebo/xmlschema/#interface">
-  <property name="M_PI" value="3.1415926535897931" />
+<robot xmlns:xacro="http://www.ros.org/wiki/xacro">
   <!--
-     Little helper macro to define the inertia matrix needed
-     for links.
-     -->
-  <macro name="cuboid_inertia_def" params="width height length mass">
+		Little helper macro to define the inertia matrix needed
+		for links.
+  -->
+  <xacro:macro name="cuboid_inertia_def" params="width height length mass">
     <inertia ixx="${mass * (height * height + length * length) / 12}"
              iyy="${mass * (width * width + length * length) / 12}"
              izz="${mass * (width * width + height * height) / 12}"
              ixy="0" iyz="0" ixz="0"/>
-  </macro>
+  </xacro:macro>
   <!-- length is along the y-axis! -->
-  <macro name="cylinder_inertia_def" params="radius length mass">
+  <xacro:macro name="cylinder_inertia_def" params="radius length mass">
     <inertia ixx="${mass * (3 * radius * radius + length * length) / 12}"
              iyy="${mass * radius*radius / 2}"
              izz="${mass * (3 * radius * radius + length * length) / 12}"
              ixy="0" iyz="0" ixz="0"/>
-  </macro>
+  </xacro:macro>
 </robot>
