Commit message: Added support for parametrized end-effector flange pose

File: lwr_description/urdf/lwr.urdf.xacro (robot description, xacro)
@@ -13,5 +13,11 @@
   <xacro:property name="joint_damping_factor" value="1.0" />
   <xacro:property name="arm_velocity_scale_factor" value="1"/>
-  <xacro:macro name="kuka_lwr_arm" params="name">
+  <xacro:macro name="kuka_lwr_arm" params="name
+                                           toolmount_x:=0
+                                           toolmount_y:=0
+                                           toolmount_z:=0.078
+                                           toolmount_yaw:=0
+                                           toolmount_pitch:=0
+                                           toolmount_roll:=0">
     <link name="${name}arm_base_link">
       <inertial>
@@ -368,4 +374,5 @@
     </gazebo>
     <joint name="${name}arm_hand_fixed_joint" type="fixed">
+      <origin xyz="${toolmount_x} ${toolmount_y} ${toolmount_z-0.078}" rpy="${toolmount_roll} ${toolmount_pitch} ${toolmount_yaw}"/>
       <parent link="${name}arm_7_link"/>
       <child link="${name}tool_mount"/>
